File: C64 Pi1541-II FaceplateB/C64 Pi1541-II FaceplateB.kicad_pcb (KiCad board)
At the start: 2 copper layers, 97.8 x 97.8 mm, 9 parts, among them IC1 0.96_OLED, J4 Faceplate, M1 Mounting, M2 Mounting, M3 Mounting, M4 Mounting

Commit message: Updated gerber files
Routing:
- net I2C_SDA: track 98.2 -> 94.7 mm, vias 2 -> 0
- net I2C_SCL: track 97.9 -> 97.2 mm, vias 2 -> 0
Other:
- rule pad_to_mask_clearance: 0.2 -> 0
