File: C64 Pi1541-II Module/C64 Pi1541-II Module.kicad_pcb (KiCad board)
At the start: 2 copper layers, 97.8 x 97.8 mm, 31 parts, among them IC1 0.96_OLED, IC2 7406, IC3 I2C LC, J1 DC IN, J2 C64_IEC, J3 C64_IEC, J4 Faceplate, M1 Mounting, M2 Mounting, M3 Mounting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

Commit message: Added copper layer to backplate
Parts:
- moved REF** 1.91 mm to (83.2, 74.4)
Other:
- board text added: "PI1541-II Module (rev. B) github.com/tebl Licensed under CERN OHL v.1.2"
- board text removed: "PI1541-II revision A github.com/tebl Licensed under CERN OHL v.1.2"
Changed lines of the file:
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@@
   (page A4)
   (layers
-    (0 F.Cu signal)
-    (31 B.Cu signal)
+    (0 F.Cu signal hide)
+    (31 B.Cu signal hide)
     (32 B.Adhes user)
     (33 F.Adhes user)
@@
   )
   (module Symbols:Symbol_Barrel_Polarity locked (layer B.Cu)
-    (at 81.28 74.422)
+    (at 83.185 74.422)
     (descr "Barrel connector polarity indicator")
     (tags "barrel polarity")
@@
     )
   )
-  (gr_text - (at 78.3336 74.3966 180) (layer B.SilkS)
+  (gr_text - (at 80.2386 74.3966 180) (layer B.SilkS)
     (effects (font (size 1 1) (thickness 0.15)) (justify mirror))
   )
@@
     (effects (font (size 1.5 1.5) (thickness 0.15)))
   )
-  (gr_text "PI1541-II revision A\ngithub.com/tebl\n\nLicensed under\nCERN OHL v.1.2" (at 138.24 102.59) (layer B.SilkS)
+  (gr_text "PI1541-II\nModule (rev. B)\ngithub.com/tebl\n\nLicensed under\nCERN OHL v.1.2" (at 138.24 102.59) (layer B.SilkS)
     (effects (font (size 1.5 1.5) (thickness 0.15)) (justify mirror))
   )
-  (gr_text + (at 84.26 74.29) (layer B.SilkS)
+  (gr_text + (at 86.165 74.29) (layer B.SilkS)
     (effects (font (size 1 1) (thickness 0.15)) (justify mirror))
   )
-  (gr_text "5V DC" (at 81.23 72.32) (layer B.SilkS)
+  (gr_text "5V DC" (at 83.135 72.32) (layer B.SilkS)
     (effects (font (size 1 1) (thickness 0.15)) (justify mirror))
   )

Commit message: Adapted some of the input from Cologran, revision C of the main module.
Parts:
- moved REF** 16.5 mm to (83.8, 57.9)
- moved R1 15.3 mm to (97.2, 78.7), turned to 90 degrees
- moved R2 15.3 mm to (118.7, 78.7), turned to 90 degrees
- moved REF** 14.1 mm to (83.8, 57.8)
- moved J1 9.86 mm to (83.8, 68.6), turned to 270 degrees
- moved REF** 5.12 mm to (74.4, 82.5)
- moved BZ1 1.00 mm to (155.9, 79.5)
Connections:
- A1 pad 10: (no net) -> Net-(A1-Pad10)
- A1 pad 17: (no net) -> Net-(A1-Pad17)
- A1 pad 19: (no net) -> Net-(A1-Pad19)
- A1 pad 21: (no net) -> Net-(A1-Pad21)
- A1 pad 23: (no net) -> Net-(A1-Pad23)
- A1 pad 24: (no net) -> Net-(A1-Pad24)
- A1 pad 26: (no net) -> Net-(A1-Pad26)
- A1 pad 27: (no net) -> Net-(A1-Pad27)
- A1 pad 28: (no net) -> Net-(A1-Pad28)
- A1 pad 31: (no net) -> Net-(A1-Pad31)
- A1 pad 32: (no net) -> Net-(A1-Pad32)
- A1 pad 35: (no net) -> Net-(A1-Pad35)
- A1 pad 4: (no net) -> Net-(A1-Pad4)
- A1 pad 40: (no net) -> Net-(A1-Pad40)
- A1 pad 8: (no net) -> Net-(A1-Pad8)
- IC2 pad 10: (no net) -> Net-(IC2-Pad10)
- IC2 pad 11: (no net) -> Net-(IC2-Pad11)
- IC2 pad 12: (no net) -> Net-(IC2-Pad12)
- IC2 pad 13: (no net) -> Net-(IC2-Pad13)
- IC2 pad 5: (no net) -> Net-(IC2-Pad5)
- IC2 pad 6: (no net) -> Net-(IC2-Pad6)
- IC2 pad 8: (no net) -> Net-(IC2-Pad8)
- IC2 pad 9: (no net) -> Net-(IC2-Pad9)
- J2 pad 1: (no net) -> Net-(J2-Pad1)
- J3 pad 1: (no net) -> Net-(J3-Pad1)
Routing:
- net +5V: track 175.8 -> 104.9 mm, vias 6 -> 3
- net C64_DATA: track 89.6 -> 95.9 mm
- net C64_CLK: track 76.5 -> 70.7 mm
- net I2C_SDA: track 138.6 -> 133.6 mm, vias 2 -> 3
- net +3V3: track 144.9 -> 149.0 mm
- net Net-(A1-Pad33): track 47.9 -> 44.4 mm
- net I2C_SCL: track 138.1 -> 135.2 mm
- net C64_RST: track 65.6 -> 63.7 mm
Other:
- outline, holes or cut-outs redrawn
- rule pad_to_mask_clearance: 0.2 -> 0
- board text added: "1. Install smaller components (resistors, capacitors etc). 2. Install logic level converter module, trim down pins to size. 3. Install 7406 socket 4. Install 40 pin Raspberry Pi header if needed, adjust to match supporting standoffs oppsite. before soldering. 5. If installing 0.96" OLED here, link JP1 and JP2 to match OLED pinouts (1-2 when GND, VCC, SCL, SDA). Use female header for added height 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"
- board text added: "PI1541-II Module (rev. C) github.com/tebl Licensed under CERN OHL v.1.2"
- board text removed: "1. Install smaller components (resistors, capacitors etc). 2. Install logic level converter module, trim down pins to size. 3. Install 7406 socket 4. Install 40 pin Raspberry Pi header if needed, adjust to match supporting standoffs oppsite. before soldering. 5. If installing 0.96" OLED here, link JP1 and JP2 to match OLED pinouts (1-2 when GND, VCC, SCL, SDA). Use female header for added height.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"
- board text removed: "PI1541-II Module (rev. B) github.com/tebl Licensed under CERN OHL v.1.2"
