File: C64 Pi1541-II Module/C64 Pi1541-II Module.sch (KiCad schematic (older format))
At the start: 27 parts, among them IC1 0.96_OLED, IC2 7406, IC3 I2C LC, J1 DC IN, J2 C64_IEC, J3 C64_IEC, J4 Faceplate, M1 Mounting, M2 Mounting, M3 Mounting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

Commit message: Adapted some of the input from Cologran, revision C of the main module.
Parts:
- A1: symbol Connector:Raspberry_Pi_2_3 -> raspberry_pi:Raspberry_Pi_2_3
- JP1, JP2: symbol Jumper:SolderJumper_3_Open -> I2C_OLED:PowerSelect
Changed lines of the file:
@@
 Connection ~ 6375 10200
 $Comp
-L Connector:Raspberry_Pi_2_3 A1
+L raspberry_pi:Raspberry_Pi_2_3 A1
 U 1 1 5EE82FB5
 P 2775 3750
@@
 I2C_SCL
 $Comp
-L Jumper:SolderJumper_3_Open JP2
+L I2C_OLED:PowerSelect JP2
 U 1 1 5F12F8C1
 P 8400 8700
@@
 $EndComp
 $Comp
-L Jumper:SolderJumper_3_Open JP1
+L I2C_OLED:PowerSelect JP1
 U 1 1 5F14C67F
 P 7800 8700
